File: PGA2320.kicad_pcb (KiCad board)
At the start: 2 copper layers, 50 x 50 mm, 24 parts, among them J3 2P-2.54, J4 3P-2.54, P1 SDO, P2 CONTROLLER, U1 PGA2320

Commit message: improvements
Parts:
- moved R1 0.51 mm to (125.5, 60.2)
- moved D1 0.51 mm to (125.5, 62.2)
Routing:
- net VOUT_R: vias 1 -> 0
- net VOUT_L: vias 1 -> 0
- net VIN_L: vias 1 -> 0
- net GND_D: vias 1 -> 4
- net GND_A: vias 2 -> 3
Changed lines of the file:
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@@
   )
   (footprint "Resistor_SMD:R_0805_2012Metric_Pad1.20x1.40mm_HandSolder" (layer "F.Cu")
-    (at 125.476 59.69)
+    (at 125.476 60.198)
     (descr "Resistor SMD 0805 (2012 Metric), square (rectangular) end terminal, IPC_7351 nominal with elongated pad for handsoldering. (Body size source: IPC-SM-782 page 72, https://www.pcb-3d.com/wordpress/wp-content/uploads/ipc-sm-782a_amendment_1_and_2.pdf), generated with kicad-footprint-generator")
     (tags "resistor handsolder")
@@
   )
   (footprint "LED_SMD:LED_0805_2012Metric_Pad1.15x1.40mm_HandSolder" (layer "F.Cu")
-    (at 125.476 61.722 180)
+    (at 125.476 62.23 180)
     (descr "LED SMD 0805 (2012 Metric), square (rectangular) end terminal, IPC_7351 nominal, (Body size source: https://docs.google.com/spreadsheets/d/1BsfQQcO9C6DZCsRaXUlFlo91Tg2WpOkGARC1WS5S8t0/edit?usp=sharing), generated with kicad-footprint-generator")
     (tags "LED handsolder")
@@
   (segment (start 136.835696 82.804) (end 136.859513 82.827817) (width 0.25) (layer "F.Cu") (net 1))
   (segment (start 128.773 59.436) (end 129.535 60.198) (width 0.25) (layer "F.Cu") (net 1))
-  (segment (start 126.476 59.436) (end 128.773 59.436) (width 0.25) (layer "F.Cu") (net 1))
+  (segment (start 126.476 59.944) (end 128.773 59.944) (width 0.25) (layer "F.Cu") (net 1))
   (segment (start 135.382 82.804) (end 136.835696 82.804) (width 0.25) (layer "F.Cu") (net 1))
   (via (at 135.382 82.804) (size 0.8) (drill 0.4) (layers "F.Cu" "B.Cu") (free) (net 1))
@@
   (segment (start 129.535 60.198) (end 129.535 79.697539) (width 0.25) (layer "B.Cu") (net 1))
   (arc (start 129.535 79.697539) (mid 129.734336 80.699672) (end 130.302 81.54924) (width 0.25) (layer "B.Cu") (net 1))
+  (via (at 131.572 78.232) (size 0.8) (drill 0.4) (layers "F.Cu" "B.Cu") (free) (net 2))
+  (via (at 131.826 71.12) (size 0.8) (drill 0.4) (layers "F.Cu" "B.Cu") (free) (net 2))
   (via (at 135.382 84.074) (size 0.8) (drill 0.4) (layers "F.Cu" "B.Cu") (free) (net 2))
+  (via (at 132.08 63.754) (size 0.8) (drill 0.4) (layers "F.Cu" "B.Cu") (free) (net 2))
   (segment (start 133.604 84.5185) (end 134.9375 84.5185) (width 0.25) (layer "B.Cu") (net 2))
   (segment (start 130.302 86.59876) (end 132.38226 84.5185) (width 0.25) (layer "B.Cu") (net 2))
@@
   (segment (start 132.38226 84.5185) (end 133.604 84.5185) (width 0.25) (layer "B.Cu") (net 2))
   (segment (start 156.217 62.713) (end 156.242 62.738) (width 0.25) (layer "F.Cu") (net 3))
+  (via (at 154.432 83.566) (size 0.8) (drill 0.4) (layers "F.Cu" "B.Cu") (free) (net 3))
   (via (at 147.828 80.264) (size 0.8) (drill 0.4) (layers "F.Cu" "B.Cu") (free) (net 3))
   (via (at 147.828 86.614) (size 0.8) (drill 0.4) (layers "F.Cu" "B.Cu") (free) (net 3))
@@
   (segment (start 146.812 67.834) (end 146.812 83.058) (width 0.25) (layer "B.Cu") (net 5))
   (segment (start 147.828 84.074) (end 148.7805 84.074) (width 0.25) (layer "B.Cu") (net 5))
-  (segment (start 124.476 59.436) (end 124.476 61.443) (width 0.25) (layer "F.Cu") (net 6))
-  (segment (start 124.476 61.443) (end 124.451 61.468) (width 0.25) (layer "F.Cu") (net 6))
+  (segment (start 124.476 59.944) (end 124.476 61.951) (width 0.25) (layer "F.Cu") (net 6))
+  (segment (start 124.476 61.951) (end 124.451 61.976) (width 0.25) (layer "F.Cu") (net 6))
   (segment (start 143.796 60.706) (end 143.796 62.976) (width 0.25) (layer "F.Cu") (net 7))
   (segment (start 143.796 62.976) (end 143.78 62.992) (width 0.25) (layer "F.Cu") (net 7))
@@
   (segment (start 160.027696 79.017817) (end 162.845513 76.2) (width 0.25) (layer "F.Cu") (net 9))
   (segment (start 146.481033 79.017817) (end 160.027696 79.017817) (width 0.25) (layer "F.Cu") (net 9))
-  (via (at 159.512 78.994) (size 0.8) (drill 0.4) (layers "F.Cu" "B.Cu") (net 9))
   (segment (start 159.488183 87.907817) (end 159.512 87.884) (width 0.25) (layer "F.Cu") (net 10))
   (segment (start 146.481033 87.907817) (end 159.488183 87.907817) (width 0.25) (layer "F.Cu") (net 10))
@@
   (segment (start 158.096484 81.557817) (end 158.496 81.957333) (width 0.25) (layer "F.Cu") (net 11))
   (segment (start 146.481033 81.557817) (end 158.096484 81.557817) (width 0.25) (layer "F.Cu") (net 11))
-  (via (at 159.512 81.957333) (size 0.8) (drill 0.4) (layers "F.Cu" "B.Cu") (free) (net 11))
+  (segment (start 161.803 90.175) (end 162.845513 90.175) (width 0.25) (layer "F.Cu") (net 12))
+  (segment (start 160.782 89.154) (end 161.803 90.175) (width 0.25) (layer "F.Cu") (net 12))
+  (segment (start 159.584894 85.367817) (end 160.782 86.564923) (width 0.25) (layer "F.Cu") (net 12))
   (segment (start 160.782 86.564923) (end 160.782 89.154) (width 0.25) (layer "F.Cu") (net 12))
-  (segment (start 159.536891 85.319814) (end 160.782 86.564923) (width 0.25) (layer "F.Cu") (net 12))
-  (segment (start 159.536891 85.319814) (end 159.488888 85.367817) (width 0.25) (layer "F.Cu") (net 12))
-  (segment (start 159.488888 85.367817) (end 146.481033 85.367817) (width 0.25) (layer "F.Cu") (net 12))
-  (segment (start 160.782 89.154) (end 161.803 90.175) (width 0.25) (layer "F.Cu") (net 12))
-  (segment (start 161.803 90.175) (end 162.845513 90.175) (width 0.25) (layer "F.Cu") (net 12))
-  (via (at 159.536891 85.319814) (size 0.8) (drill 0.4) (layers "F.Cu" "B.Cu") (free) (net 12))
+  (segment (start 146.481033 85.367817) (end 159.584894 85.367817) (width 0.25) (layer "F.Cu") (net 12))
   (segment (start 138.660183 86.637817) (end 138.684 86.614) (width 0.25) (layer "F.Cu") (net 13))
   (segment (start 136.859513 86.637817) (end 138.660183 86.637817) (width 0.25) (layer "F.Cu") (net 13))
@@
   (segment (start 135.382 81.534) (end 136.835696 81.534) (width 0.25) (layer "F.Cu") (net 16))
   (via (at 135.382 81.534) (size 0.8) (drill 0.4) (layers "F.Cu" "B.Cu") (free) (net 16))
-  (segment (start 134.207 81.121) (end 134.62 81.534) (width 0.25) (layer "B.Cu") (net 16))
-  (segment (start 134.207 68.485) (end 134.207 81.121) (width 0.25) (layer "B.Cu") (net 16))
-  (segment (start 137.414 65.278) (end 134.207 68.485) (width 0.25) (layer "B.Cu") (net 16))
   (segment (start 134.62 81.534) (end 135.382 81.534) (width 0.25) (layer "B.Cu") (net 16))
+  (segment (start 133.858 80.772) (end 134.62 81.534) (width 0.25) (layer "B.Cu") (net 16))
+  (segment (start 133.858 68.834) (end 133.858 80.772) (width 0.25) (layer "B.Cu") (net 16))
+  (segment (start 137.414 65.278) (end 133.858 68.834) (width 0.25) (layer "B.Cu") (net 16))
   (segment (start 136.859513 85.367817) (end 138.660183 85.367817) (width 0.25) (layer "F.Cu") (net 17))
   (segment (start 138.660183 85.367817) (end 138.684 85.344) (width 0.25) (layer "F.Cu") (net 17))
   (via (at 138.684 85.344) (size 0.8) (drill 0.4) (layers "F.Cu" "B.Cu") (free) (net 17))
-  (segment (start 138.684 64.54902) (end 138.684 85.344) (width 0.25) (layer "B.Cu") (net 17))
-  (segment (start 137.414 63.27902) (end 138.684 64.54902) (width 0.25) (layer "B.Cu") (net 17))
+  (segment (start 139.192 65.05702) (end 139.192 84.836) (width 0.25) (layer "B.Cu") (net 17))
+  (segment (start 137.414 63.27902) (end 139.192 65.05702) (width 0.25) (layer "B.Cu") (net 17))
+  (segment (start 139.192 84.836) (end 138.684 85.344) (width 0.25) (layer "B.Cu") (net 17))
   (segment (start 138.660183 87.907817) (end 138.684 87.884) (width 0.25) (layer "F.Cu") (net 18))
   (segment (start 136.859513 87.907817) (end 138.660183 87.907817) (width 0.25) (layer "F.Cu") (net 18))
   (via (at 138.684 87.884) (size 0.8) (drill 0.4) (layers "F.Cu" "B.Cu") (free) (net 18))
-  (segment (start 139.409 87.159) (end 138.684 87.884) (width 0.25) (layer "B.Cu") (net 18))
-  (segment (start 139.409 63.2725) (end 139.409 87.159) (width 0.25) (layer "B.Cu") (net 18))
-  (segment (start 137.414 61.2775) (end 139.409 63.2725) (width 0.25) (layer "B.Cu") (net 18))
+  (segment (start 137.414 61.2775) (end 139.954 63.8175) (width 0.25) (layer "B.Cu") (net 18))
+  (segment (start 139.954 86.614) (end 138.684 87.884) (width 0.25) (layer "B.Cu") (net 18))
+  (segment (start 139.954 63.8175) (end 139.954 86.614) (width 0.25) (layer "B.Cu") (net 18))
   (zone (net 3) (net_name "GND_A") (layers "F&B.Cu") (hatch edge 0.5)
     (connect_pads (clearance 0.5))
