File: PGA2320.kicad_pcb (KiCad board)
At the start: 2 copper layers, 50 x 50 mm, 24 parts, among them J3 2P-2.54, J4 3P-2.54, P1 SDO, P2 CONTROLLER, U1 PGA2320

Commit message: improvements
Parts:
- C3, C4, C5, C6: moved to F.Cu
- P1: value SDO -> SDO_TO_OTHER_PGA2311
- moved C5 0.51 mm to (154.9, 81.5)
- moved C6 0.51 mm to (154.9, 85.3)
- moved C3 0.51 mm to (149.6, 81.5)
- moved C4 0.51 mm to (149.6, 85.3)
- renumbered IN to J1, OUT to J2
Routing:
- net GND_A: track 2.84 -> 25.4 mm, vias 3 -> 1
- net VOUT_L: track 17.8 -> 26.3 mm, vias 0 -> 2
- net +15V: track 32.7 -> 38.2 mm
- net -15V: track 29.5 -> 32.0 mm
- net VOUT_R: track 19.9 -> 20.6 mm, vias 0 -> 2
- net VIN_R: track 21.2 -> 21.7 mm, vias 1 -> 0

Commit message: improvements
Routing:
- net VOUT_R: track 20.6 -> 23.6 mm
- net VOUT_L: track 26.3 -> 27.3 mm
Changed lines of the file:
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@@
   (arc (start 160.274 82.55) (mid 160.645974 81.651974) (end 161.544 81.28) (width 0.25) (layer "F.Cu") (net 10))
   (segment (start 162.56 81.28) (end 162.845513 81.28) (width 0.25) (layer "B.Cu") (net 10))
+  (segment (start 150.368 90.17) (end 159.034369 90.17) (width 0.25) (layer "F.Cu") (net 11))
+  (segment (start 159.034369 90.17) (end 161.038434 88.165935) (width 0.25) (layer "F.Cu") (net 11))
   (segment (start 161.038434 88.165935) (end 161.038434 86.006665) (width 0.25) (layer "F.Cu") (net 11))
-  (segment (start 149.606 89.154) (end 160.050369 89.154) (width 0.25) (layer "F.Cu") (net 11))
   (segment (start 162.047 85.095) (end 162.845513 85.095) (width 0.25) (layer "F.Cu") (net 11))
   (segment (start 146.481033 81.557817) (end 148.058183 81.557817) (width 0.25) (layer "F.Cu") (net 11))
-  (segment (start 160.050369 89.154) (end 161.038434 88.165935) (width 0.25) (layer "F.Cu") (net 11))
   (segment (start 148.058183 81.557817) (end 148.082 81.534) (width 0.25) (layer "F.Cu") (net 11))
   (via (at 148.082 81.534) (size 0.8) (drill 0.4) (layers "F.Cu" "B.Cu") (free) (net 11))
-  (via (at 149.606 89.154) (size 0.8) (drill 0.4) (layers "F.Cu" "B.Cu") (free) (net 11))
+  (via (at 150.368 90.17) (size 0.8) (drill 0.4) (layers "F.Cu" "B.Cu") (free) (net 11))
   (arc (start 161.038434 86.006665) (mid 161.368054 85.356898) (end 162.047 85.095) (width 0.25) (layer "F.Cu") (net 11))
-  (segment (start 149.606 83.058) (end 149.606 89.154) (width 0.25) (layer "B.Cu") (net 11))
-  (arc (start 148.082 81.534) (mid 149.159631 81.980369) (end 149.606 83.058) (width 0.25) (layer "B.Cu") (net 11))
+  (segment (start 150.368 90.17) (end 149.606 89.408) (width 0.25) (layer "B.Cu") (net 11))
+  (segment (start 149.606 89.408) (end 149.606 83.058) (width 0.25) (layer "B.Cu") (net 11))
+  (arc (start 149.606 83.058) (mid 149.159631 81.980369) (end 148.082 81.534) (width 0.25) (layer "B.Cu") (net 11))
   (segment (start 146.481033 85.367817) (end 148.058183 85.367817) (width 0.25) (layer "F.Cu") (net 12))
-  (segment (start 148.082 89.154) (end 149.098 90.17) (width 0.25) (layer "F.Cu") (net 12))
-  (segment (start 149.098 90.17) (end 162.840513 90.17) (width 0.25) (layer "F.Cu") (net 12))
+  (segment (start 160.808513 92.202) (end 162.840513 90.17) (width 0.25) (layer "F.Cu") (net 12))
+  (segment (start 148.336 91.694) (end 148.844 92.202) (width 0.25) (layer "F.Cu") (net 12))
+  (segment (start 148.844 92.202) (end 160.808513 92.202) (width 0.25) (layer "F.Cu") (net 12))
   (segment (start 148.058183 85.367817) (end 148.082 85.344) (width 0.25) (layer "F.Cu") (net 12))
-  (via (at 148.082 89.154) (size 0.8) (drill 0.4) (layers "F.Cu" "B.Cu") (free) (net 12))
+  (via (at 148.336 91.694) (size 0.8) (drill 0.4) (layers "F.Cu" "B.Cu") (free) (net 12))
   (via (at 148.082 85.344) (size 0.8) (drill 0.4) (layers "F.Cu" "B.Cu") (free) (net 12))
   (arc (start 162.840513 90.17) (mid 162.844049 90.17146) (end 162.845513 90.175) (width 0.25) (layer "F.Cu") (net 12))
-  (segment (start 148.082 85.344) (end 148.082 89.154) (width 0.25) (layer "B.Cu") (net 12))
+  (segment (start 148.336 91.694) (end 148.082 91.44) (width 0.25) (layer "B.Cu") (net 12))
+  (segment (start 148.082 91.44) (end 148.082 85.344) (width 0.25) (layer "B.Cu") (net 12))
   (segment (start 138.660183 86.637817) (end 138.684 86.614) (width 0.25) (layer "F.Cu") (net 13))
   (segment (start 136.859513 86.637817) (end 138.660183 86.637817) (width 0.25) (layer "F.Cu") (net 13))

Commit message: improvements
Parts:
- added C7: 100pf, Capacitor_SMD:C_0805_2012Metric, F.Cu at (203.6, 74.2)
- added Q1: BC550, Package_TO_SOT_THT:TO-92_Inline, F.Cu at (188.8, 74.4)
- added Q2: BC560, Package_TO_SOT_THT:TO-92_Inline, F.Cu at (194.6, 74.4)
- added R4: 1k, Resistor_SMD:R_0805_2012Metric_Pad1.20x1.40mm_HandSolder, F.Cu at (187.0, 78.8)
- added R5: 1k, Resistor_SMD:R_0805_2012Metric_Pad1.20x1.40mm_HandSolder, F.Cu at (189.9, 78.8)
- added R6: 25k, Resistor_SMD:R_0805_2012Metric_Pad1.20x1.40mm_HandSolder, F.Cu at (192.9, 78.8)
- added R7: 5k, Resistor_SMD:R_0805_2012Metric_Pad1.20x1.40mm_HandSolder, F.Cu at (195.8, 78.8)
- added R8: 5k, Resistor_SMD:R_0805_2012Metric_Pad1.20x1.40mm_HandSolder, F.Cu at (198.8, 78.8)
- added R9: 26.2k, Resistor_SMD:R_0805_2012Metric_Pad1.20x1.40mm_HandSolder, F.Cu at (201.7, 78.8)
- added VR1: TL431AIDBZR, digikey-footprints:SOT-23-3, F.Cu at (199.6, 74.1)
- added VR2: TL431AIDBZR, digikey-footprints:SOT-23-3, F.Cu at (199.6, 69.4)

Commit message: psu payout
Parts:
- moved C7 58.6 mm to (145.0, 76.9), turned to -90 degrees
- moved VR1 50.8 mm to (148.8, 72.9), turned to 0 degrees
- moved R7 48.3 mm to (147.5, 77.0), turned to -90 degrees
- moved Q1 43.1 mm to (146.1, 68.8), turned to 0 degrees
- moved R9 43.1 mm to (158.7, 77.0)
- moved R8 42.9 mm to (155.9, 77.0), turned to -90 degrees
- moved R6 42.9 mm to (150.1, 77.0)
- moved R4 42.4 mm to (145.0, 72.9), turned to -90 degrees
- moved VR2 40.5 mm to (159.3, 73.0), turned to 180 degrees
- moved Q2 38.0 mm to (157.0, 68.9), turned to 0 degrees
- moved R5 34.5 mm to (155.9, 73.0), turned to -90 degrees
- moved C4 7.34 mm to (149.6, 92.7)
- moved C6 7.34 mm to (154.9, 92.7)
- moved J2 7.34 mm to (162.8, 92.4)
- moved JP1 7.34 mm to (146.7, 102.6)
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Connections:
- D3 pad 1: -15V -> /-16V to -18V
- J4 pad 1: +15V -> /+16V to +18V
- J4 pad 3: -15V -> /-16V to -18V
- Q1 pad 1: Net-(Q1-C) -> /+16V to +18V
- Q2 pad 1: Net-(Q2-C) -> /-16V to -18V
- R2 pad 1: +15V -> /+16V to +18V
- R4 pad 1: Net-(Q1-C) -> /+16V to +18V
- R5 pad 1: Net-(Q2-C) -> /-16V to -18V
Routing:
- net /-16V to -18V: track 0.00 -> 15.0 mm
- net /+16V to +18V: track 0.00 -> 13.9 mm
- net Net-(VR2-REF): track 0.00 -> 10.9 mm
- net Net-(Q2-B): track 0.00 -> 9.30 mm
- net Net-(Q1-B): track 0.00 -> 8.93 mm
- net Net-(VR1-REF): track 0.00 -> 8.13 mm
- net -15V: track 32.0 -> 35.9 mm
- net +15V: track 38.2 -> 39.8 mm

Commit message: add PI filter
Parts:
- added C10: 10uf, Capacitor_SMD:C_0805_2012Metric, F.Cu at (173.0, 72.4)
- added C11: 10uf, Capacitor_SMD:C_0805_2012Metric, F.Cu at (173.0, 75.4)
- added C8: 10uf, Capacitor_SMD:C_0805_2012Metric, F.Cu at (146.0, 80.3)
- added C9: 10uf, Capacitor_SMD:C_0805_2012Metric, F.Cu at (146.0, 82.8)
- added L1: 47uH, Inductor_SMD:L_0805_2012Metric, F.Cu at (153.2, 81.5)
- added L2: 47uH, Inductor_SMD:L_0805_2012Metric, F.Cu at (177.5, 74.9)
- added R10: 10, Resistor_SMD:R_0805_2012Metric_Pad1.20x1.40mm_HandSolder, F.Cu at (149.9, 81.3)
- added R11: 10, Resistor_SMD:R_0805_2012Metric_Pad1.20x1.40mm_HandSolder, F.Cu at (177.6, 69.3)
Connections:
- Q1 pad 3: +15V -> Net-(Q1-E)
- Q2 pad 3: -15V -> Net-(Q2-E)
- R6 pad 1: +15V -> Net-(Q1-E)

Commit message: improvements
Parts:
- moved L2 22.2 mm to (155.7, 79.0), turned to 180 degrees
- moved R11 20.5 mm to (159.5, 79.0), turned to 180 degrees
- moved C11 18.2 mm to (155.7, 81.1), turned to 180 degrees
- moved C10 16.2 mm to (159.3, 81.1)
- moved L1 7.92 mm to (145.6, 79.3), turned to 180 degrees
- moved C8 3.37 mm to (149.2, 81.3)
- moved R10 2.07 mm to (149.4, 79.3), turned to 180 degrees
- moved R7 1.95 mm to (148.3, 75.2), turned to 0 degrees
- moved R6 1.74 mm to (148.4, 77.3), turned to 180 degrees
- moved C9 1.54 mm to (145.6, 81.3), turned to 180 degrees
- moved Q2 1.22 mm to (156.2, 68.0)
- moved R5 1.22 mm to (155.2, 72.0)
- moved R8 1.22 mm to (155.2, 76.1)
- moved R9 1.22 mm to (158.0, 76.1)
- moved VR2 1.22 mm to (158.5, 72.0)
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Routing:
- net Net-(Q1-E): track 0.00 -> 17.4 mm
- net -15V: track 35.9 -> 18.6 mm
- net Net-(Q2-E): track 0.00 -> 15.8 mm
- net +15V: track 39.8 -> 27.4 mm
- net GND_A: track 25.4 -> 28.7 mm, vias 1 -> 3
- net Net-(L1-Pad1): track 0.00 -> 2.48 mm
- net Net-(L2-Pad1): track 0.00 -> 1.75 mm
- net Net-(VR1-REF): track 8.13 -> 6.88 mm
- net /-16V to -18V: track 15.0 -> 13.9 mm
- net VIN_R: track 21.7 -> 20.8 mm
- net Net-(Q1-B): track 8.93 -> 8.15 mm

Commit message: improvements
Parts:
- moved C1 7.47 mm to (133.6, 91.0)
- moved C2 7.44 mm to (129.6, 91.5)
Routing:
- net ZCEN: track 12.0 -> 19.4 mm
- net CS: track 15.9 -> 23.3 mm
- net SDO: track 16.6 -> 23.9 mm
- net +5VD: track 32.0 -> 39.3 mm
- net MUTE: track 30.0 -> 37.2 mm
- net SCLK: track 24.8 -> 31.8 mm
- net SDI: track 20.3 -> 27.2 mm
- net GND_D: track 6.13 -> 6.81 mm

Commit message: improvements
Routing:
- net Net-(VR1-REF): track 6.88 -> 6.32 mm
Changed lines of the file:
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@@
   (segment (start 145 72.956) (end 145 75.02) (width 0.5) (layer "F.Cu") (net 19))
   (segment (start 147.32 70.684) (end 147.032 70.972) (width 0.5) (layer "F.Cu") (net 19))
-  (segment (start 147.3455 74.716) (end 147.3455 76.986) (width 0.5) (layer "F.Cu") (net 20))
-  (segment (start 147.252 72.872) (end 147.252 74.6225) (width 0.5) (layer "F.Cu") (net 20))
-  (segment (start 147.54 73.076) (end 147.76 72.856) (width 0.5) (layer "F.Cu") (net 20))
-  (segment (start 147.252 74.6225) (end 147.3455 74.716) (width 0.5) (layer "F.Cu") (net 20))
+  (segment (start 145.082 77.002) (end 145 76.92) (width 0.5) (layer "F.Cu") (net 20))
+  (segment (start 147.3455 73.2195) (end 147.3455 76.986) (width 0.5) (layer "F.Cu") (net 20))
+  (segment (start 147.252 73.126) (end 147.3455 73.2195) (width 0.5) (layer "F.Cu") (net 20))
+  (segment (start 147.3455 76.986) (end 147.3615 77.002) (width 0.5) (layer "F.Cu") (net 20))
   (segment (start 147.3615 77.002) (end 145.082 77.002) (width 0.5) (layer "F.Cu") (net 20))
-  (segment (start 145.082 77.002) (end 145 76.92) (width 0.5) (layer "F.Cu") (net 20))
-  (segment (start 147.3455 76.986) (end 147.3615 77.002) (width 0.5) (layer "F.Cu") (net 20))
   (segment (start 156.1855 71.988) (end 155.1855 72.988) (width 0.5) (layer "F.Cu") (net 21))
   (segment (start 157.5055 71.802) (end 157.6915 71.988) (width 0.5) (layer "F.Cu") (net 21))
