File: PGA2320.kicad_sch (KiCad schematic)
At the start: 31 parts, among them J1 XH2.54-3P, J2 XH2.54-3P, J3 2P-2.54, J4 3P-2.54, P1 SDO_TO_OTHER_PGA2311, P2 CONTROLLER, Q1 BC550, Q2 BC560, U1 PGA2320

Commit message: psu payout
Connections:
- net +15V: no longer J4.1 (Pin_1), R2.1
- net -15V: no longer D3.1 (K), J4.3 (Pin_3)
- net +16v to +18v renamed +16V to +18V
- net +16V to +18V: now also J4.1 (Pin_1), R2.1
- net -16v to -18v renamed -16V to -18V
- net -16V to -18V: now also D3.1 (K), J4.3 (Pin_3)
Changed lines of the file:
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@@
     (stroke (width 0) (type default))
   )
-  (wire (pts (xy 264.16 111.76) (xy 266.7 111.76))
+  (wire (pts (xy 252.73 111.76) (xy 266.7 111.76))
     (stroke (width 0) (type default))
   )
@@
     (stroke (width 0) (type default))
   )
-  (wire (pts (xy 255.27 114.3) (xy 266.7 114.3))
+  (wire (pts (xy 252.73 114.3) (xy 266.7 114.3))
     (stroke (width 0) (type default))
   )
@@
     (stroke (width 0) (type default))
   )
-  (wire (pts (xy 40.64 66.04) (xy 43.18 66.04))
+  (wire (pts (xy 30.48 66.04) (xy 43.18 66.04))
     (stroke (width 0) (type default))
   )
@@
     (stroke (width 0) (type default))
   )
-  (wire (pts (xy 264.16 116.84) (xy 266.7 116.84))
+  (wire (pts (xy 252.73 116.84) (xy 266.7 116.84))
     (stroke (width 0) (type default))
   )
@@
     (effects (font (size 1.524 1.524) (thickness 0.3048) bold) (justify left bottom))
   )
-  (label "-16v to -18v" (at 21.59 170.18 0) (fields_autoplaced)
+  (label "+16V to +18V" (at 252.73 111.76 0) (fields_autoplaced)
+    (effects (font (size 1.27 1.27)) (justify left bottom))
+  )
+  (label "-16V to -18V" (at 252.73 116.84 0) (fields_autoplaced)
+    (effects (font (size 1.27 1.27)) (justify left bottom))
+  )
+  (label "-16V to -18V" (at 21.59 170.18 0) (fields_autoplaced)
+    (effects (font (size 1.27 1.27)) (justify left bottom))
+  )
+  (label "-16V to -18V" (at 64.77 77.47 0) (fields_autoplaced)
+    (effects (font (size 1.27 1.27)) (justify left bottom))
+  )
+  (label "GND_A" (at 252.73 114.3 0) (fields_autoplaced)
+    (effects (font (size 1.27 1.27)) (justify left bottom))
+  )
+  (label "+16V to +18V" (at 30.48 66.04 0) (fields_autoplaced)
     (effects (font (size 1.27 1.27)) (justify left bottom))
   )
@@
     (effects (font (size 1.27 1.27)) (justify left bottom))
   )
-  (label "+16v to +18v" (at 21.59 143.51 0) (fields_autoplaced)
+  (label "+16V to +18V" (at 21.59 143.51 0) (fields_autoplaced)
     (effects (font (size 1.27 1.27)) (justify left bottom))
   )
@@
     )
   )
-  (global_label "GND_A" (shape input) (at 255.27 114.3 180) (fields_autoplaced)
-    (effects (font (size 1.524 1.524)) (justify right))
-    (property "Intersheetrefs" "${INTERSHEET_REFS}" (at 34.925 -28.575 0)
-      (effects (font (size 1.27 1.27)) hide)
-    )
-  )
   (global_label "MUTE" (shape input) (at 168.91 58.42 180) (fields_autoplaced)
     (effects (font (size 1.524 1.524)) (justify right))
@@
     )
   )
-  (global_label "+15V" (shape input) (at 40.64 66.04 180) (fields_autoplaced)
-    (effects (font (size 1.524 1.524)) (justify right))
-    (property "Intersheetrefs" "${INTERSHEET_REFS}" (at 31.7551 65.9448 0)
-      (effects (font (size 1.524 1.524)) (justify right) hide)
-    )
-  )
   (global_label "VOUT_L" (shape input) (at 157.48 119.38 180) (fields_autoplaced)
     (effects (font (size 1.524 1.524)) (justify right))
@@
     )
   )
-  (global_label "-15V" (shape input) (at 64.77 77.47 0) (fields_autoplaced)
-    (effects (font (size 1.524 1.524)) (justify left))
-    (property "Intersheetrefs" "${INTERSHEET_REFS}" (at 73.6549 77.3748 0)
-      (effects (font (size 1.524 1.524)) (justify left) hide)
-    )
-  )
   (global_label "VOUT_R" (shape input) (at 157.48 114.3 180) (fields_autoplaced)
     (effects (font (size 1.524 1.524)) (justify right))
@@
     )
   )
-  (global_label "+15V" (shape input) (at 264.16 111.76 180) (fields_autoplaced)
-    (effects (font (size 1.524 1.524)) (justify right))
-    (property "Intersheetrefs" "${INTERSHEET_REFS}" (at 255.2751 111.6648 0)
-      (effects (font (size 1.524 1.524)) (justify right) hide)
-    )
-  )
   (global_label "GND_A" (shape input) (at 146.05 116.84 180) (fields_autoplaced)
     (effects (font (size 1.524 1.524)) (justify right))
@@
     )
   )
-  (global_label "-15V" (shape input) (at 264.16 116.84 180) (fields_autoplaced)
-    (effects (font (size 1.524 1.524)) (justify right))
-    (property "Intersheetrefs" "${INTERSHEET_REFS}" (at 255.2751 116.7448 0)
-      (effects (font (size 1.524 1.524)) (justify right) hide)
-    )
-  )

Commit message: add PI filter
Parts:
- added C10, C11, C8, C9: 10uf, Capacitor_SMD:C_0805_2012Metric, symbol Device:C
- added L1, L2: 47uH, Inductor_SMD:L_0805_2012Metric, symbol Device:L
- added R10, R11: 10, Resistor_SMD:R_0805_2012Metric_Pad1.20x1.40mm_HandSolder, symbol Device:R
Connections:
- net +15V: now also C9.2, L1.2; no longer Q1.3 (E), R6.1
- net -15V: now also C11.2, L2.2; no longer Q2.3 (E)
- net GND_A: now also C10.1, C11.1, C8.1, C9.1
- new net: C10.2, Q2.3 (E), R11.1
- new net: C8.2, Q1.3 (E), R10.1, R6.1
- new net: L1.1, R10.2
- new net: L2.1, R11.2
